Commit message: feat: add physical prop

File: src/robot_describes/urdf/xbot/base.urdf.xacro (robot description, xacro)
@@ -1,5 +1,8 @@
 <?xml version="1.0"?>
 <robot xmlns:xacro="http://www.ros.org/wiki/xacro">
+  <xacro:include filename="$(find robot_describes)/urdf/xbot/common_inertia.xacro"/>
   <xacro:macro name="base_xacro" params="length radius">
+    <!-- 虚拟部件 -->
+    <link name="base_footprint_link"/>
     <!-- 机器人身体部分 -->
     <link name="base_link">
@@ -18,5 +21,24 @@
         </material>
       </visual>
+      <collision>
+        <!-- 沿着自己几何中心的偏移和旋转 -->
+        <origin xyz="0.0 0.0 0.0" rpy="0.0 0.0 0.0"/>
+        <!-- 几何形状 -->
+        <geometry>
+          <!-- 圆柱体 -->
+          <cylinder radius="${radius}" length="${length}"/>
+        </geometry>
+        <!-- 材质和颜色 -->
+        <material name="white">
+          <color rgba="1.0 1.0 1.0 0.5" />
+        </material>
+      </collision>
+      <xacro:cylinder_inertia m="1.0" r="${radius}" h="${length}"/>
     </link>
+    <joint name="base_footprint_joint" type="fixed">
+      <parent link="base_footprint_link"/>
+      <child link="base_link"/>
+      <origin xyz="0.0 0.0 ${length / 2.0 + 0.032 - 0.001}" rpy="0.0 0.0 0.0"/>
+    </joint>
   </xacro:macro>
 </robot>

File: src/robot_describes/urdf/xbot/sensor/camera.urdf.xacro (robot description, xacro)
@@ -1,4 +1,5 @@
 <?xml version="1.0"?>
 <robot xmlns:xacro="http://www.ros.org/wiki/xacro">
+  <xacro:include filename="$(find robot_describes)/urdf/xbot/common_inertia.xacro"/>
   <xacro:macro name="camera_xacro" params="xyz">
     <link name="camera_link">
@@ -12,4 +13,14 @@
         </material>
       </visual>
+      <collision>
+        <origin xyz="0.0 0.0 0.0" rpy="0.0 0.0 0.0"/>
+        <geometry>
+          <box size="0.02 0.10 0.02" />
+        </geometry>
+        <material name="black">
+          <color rgba="0.0 0.0 0.0 1.0" />
+        </material>
+      </collision>
+      <xacro:box_inertia m="0.1" w="0.02" h="0.10" d="0.02"/>
     </link>
     <joint name="camera_joint" type="fixed">

File: src/robot_describes/urdf/xbot/sensor/imu.urdf.xacro (robot description, xacro)
@@ -1,4 +1,5 @@
 <?xml version="1.0"?>
 <robot xmlns:xacro="http://www.ros.org/wiki/xacro">
+  <xacro:include filename="$(find robot_describes)/urdf/xbot/common_inertia.xacro"/>
   <xacro:macro name="imu_xacro" params="xyz">
     <!-- 机器人的 IMU ，惯性测量单元 -->
@@ -16,4 +17,16 @@
         </material>
       </visual>
+      <collision>
+        <origin xyz="0.0 0.0 0.0" rpy="0.0 0.0 0.0"/>
+        <geometry>
+          <!-- 正方体 -->
+          <box size="0.02 0.02 0.02" />
+        </geometry>
+        <!-- 材质和颜色 -->
+        <material name="black">
+          <color rgba="0.0 0.0 0.0 1.0" />
+        </material>
+      </collision>
+      <xacro:box_inertia m="0.05" w="0.02" h="0.02" d="0.02"/>
     </link>
     <!-- 机器人关节，用来组合机器人部件 -->

File: src/robot_describes/urdf/xbot/sensor/laser.urdf.xacro (robot description, xacro)
@@ -1,4 +1,5 @@
 <?xml version="1.0"?>
 <robot xmlns:xacro="http://www.ros.org/wiki/xacro">
+  <xacro:include filename="$(find robot_describes)/urdf/xbot/common_inertia.xacro"/>
   <xacro:macro name="laser_xacro" params="xyz">
     <!-- 雷达支撑杆 -->
@@ -13,4 +14,14 @@
         </material>
       </visual>
+      <collision>
+        <origin xyz="0.0 0.0 0.0" rpy="0.0 0.0 0.0"/>
+        <geometry>
+          <cylinder radius="0.01" length="0.10" />
+        </geometry>
+        <material name="black">
+          <color rgba="0.0 0.0 0.0 1.0" />
+        </material>
+      </collision>
+      <xacro:cylinder_inertia m="0.05" r="0.01" h="0.10"/>
     </link>
     <!-- 雷达 -->
@@ -25,4 +36,14 @@
         </material>
       </visual>
+      <collision>
+        <origin xyz="0.0 0.0 0.0" rpy="0.0 0.0 0.0"/>
+        <geometry>
+          <cylinder radius="0.02" length="0.02" />
+        </geometry>
+        <material name="black">
+          <color rgba="0.0 0.0 0.0 1.0" />
+        </material>
+      </collision>
+      <xacro:cylinder_inertia m="0.10" r="0.02" h="0.02"/>
     </link>
     <joint name="laser_joint" type="fixed">

File: src/robot_describes/urdf/xbot/xbot.urdf.xacro (robot description, xacro)
@@ -1,11 +1,20 @@
 <?xml version="1.0"?>
 <robot xmlns:xacro="http://www.ros.org/wiki/xacro" name="xbot">
+  <!-- 基础部分 -->
   <xacro:include filename="$(find robot_describes)/urdf/xbot/base.urdf.xacro"/>
+  <!-- 传感器 -->
   <xacro:include filename="$(find robot_describes)/urdf/xbot/sensor/imu.urdf.xacro"/>
   <xacro:include filename="$(find robot_describes)/urdf/xbot/sensor/camera.urdf.xacro"/>
   <xacro:include filename="$(find robot_describes)/urdf/xbot/sensor/laser.urdf.xacro"/>
+  <!-- 执行器 -->
+  <xacro:include filename="$(find robot_describes)/urdf/xbot/actuator/wheel.urdf.xacro"/>
+  <xacro:include filename="$(find robot_describes)/urdf/xbot/actuator/caster.urdf.xacro"/>
   <xacro:base_xacro length="0.12" radius="0.10" />
   <xacro:imu_xacro xyz="0.0 0.0 0.02"/>
   <xacro:camera_xacro xyz="0.10 0.0 0.075"/>
   <xacro:laser_xacro xyz="0.0 0.0 0.10"/>
+  <xacro:wheel_xacro wheel_name="left_wheel" xyz="0.0 0.10 -0.06"/>
+  <xacro:wheel_xacro wheel_name="right_wheel" xyz="0.0 -0.10 -0.06"/>
+  <xacro:caster_xacro caster_name="front_caster" xyz="0.08 0 -0.076"/>
+  <xacro:caster_xacro caster_name="back_caster" xyz="-0.08 0 -0.076"/>
 </robot>
