Commit message: feat: add sensor

File: src/robot_describes/urdf/xbot/actuator/caster.urdf.xacro (robot description, xacro)
@@ -34,4 +34,14 @@
       <origin xyz="${xyz}" rpy="0.0 0.0 0.0"/>
     </joint>
+    <gazebo reference="${caster_name}_link">
+      <!-- 切向摩擦系数 -->
+      <mu1 value="0.0"/>
+      <!-- 法向摩擦系数 -->
+      <mu2 value="0.0"/>
+      <!-- 刚度系数 -->
+      <kp value="1000000000.0"/>
+      <!-- 阻尼系数 -->
+      <kd value="1.0"/>
+    </gazebo>
   </xacro:macro>
 </robot>

File: src/robot_describes/urdf/xbot/actuator/wheel.urdf.xacro (robot description, xacro)
@@ -39,4 +39,14 @@
       <axis xyz="0 1 0"/>
     </joint>
+    <gazebo reference="${wheel_name}_link">
+      <!-- 切向摩擦系数 -->
+      <mu1 value="20.0"/>
+      <!-- 法向摩擦系数 -->
+      <mu2 value="20.0"/>
+      <!-- 刚度系数 -->
+      <kp value="1000000000.0"/>
+      <!-- 阻尼系数 -->
+      <kd value="1.0"/>
+    </gazebo>
   </xacro:macro>
 </robot>

File: src/robot_describes/urdf/xbot/base.urdf.xacro (robot description, xacro)
@@ -4,5 +4,5 @@
   <xacro:macro name="base_xacro" params="length radius">
     <!-- 虚拟部件 -->
-    <link name="base_footprint_link"/>
+    <link name="base_footprint"/>
     <!-- 机器人身体部分 -->
     <link name="base_link">
@@ -37,5 +37,5 @@
     </link>
     <joint name="base_footprint_joint" type="fixed">
-      <parent link="base_footprint_link"/>
+      <parent link="base_footprint"/>
       <child link="base_link"/>
       <origin xyz="0.0 0.0 ${length / 2.0 + 0.032 - 0.001}" rpy="0.0 0.0 0.0"/>

File: src/robot_describes/urdf/xbot/sensor/camera.urdf.xacro (robot description, xacro)
@@ -9,6 +9,6 @@
           <box size="0.02 0.10 0.02" />
         </geometry>
-        <material name="black">
-          <color rgba="0.0 0.0 0.0 1.0" />
+        <material name="green">
+          <color rgba="0.0 1.0 0.0 1.0" />
         </material>
       </visual>
@@ -18,6 +18,6 @@
           <box size="0.02 0.10 0.02" />
         </geometry>
-        <material name="black">
-          <color rgba="0.0 0.0 0.0 1.0" />
+        <material name="green">
+          <color rgba="0.0 1.0 0.0 1.0" />
         </material>
       </collision>

File: src/robot_describes/urdf/xbot/sensor/laser.urdf.xacro (robot description, xacro)
@@ -32,6 +32,6 @@
           <cylinder radius="0.02" length="0.02" />
         </geometry>
-        <material name="black">
-          <color rgba="0.0 0.0 0.0 1.0" />
+        <material name="red">
+          <color rgba="1.0 0.0 0.0 1.0" />
         </material>
       </visual>
@@ -41,6 +41,6 @@
           <cylinder radius="0.02" length="0.02" />
         </geometry>
-        <material name="black">
-          <color rgba="0.0 0.0 0.0 1.0" />
+        <material name="red">
+          <color rgba="1.0 0.0 0.0 1.0" />
         </material>
       </collision>

File: src/robot_describes/urdf/xbot/xbot.urdf.xacro (robot description, xacro)
@@ -10,4 +10,6 @@
   <xacro:include filename="$(find robot_describes)/urdf/xbot/actuator/wheel.urdf.xacro"/>
   <xacro:include filename="$(find robot_describes)/urdf/xbot/actuator/caster.urdf.xacro"/>
+  <!-- 插件 -->
+  <xacro:include filename="$(find robot_describes)/urdf/xbot/plugins/gazebo_control_plugin.xacro"/>
   <xacro:base_xacro length="0.12" radius="0.10" />
   <xacro:imu_xacro xyz="0.0 0.0 0.02"/>
@@ -18,3 +20,4 @@
   <xacro:caster_xacro caster_name="front_caster" xyz="0.08 0 -0.076"/>
   <xacro:caster_xacro caster_name="back_caster" xyz="-0.08 0 -0.076"/>
+  <xacro:gazebo_control_plugin/>
 </robot>
